File: drawings/eagle/module.brd (EAGLE design)
At the start: 60.6 x 80 mm, 25 parts, among them T1 2N3904, T2 2N3904

Commit message: Finished rev1 of the circuit board and moved to a drawings directory
Parts:
- D3: value (none) -> blue; device SparkFun-LED:LED_5MM -> SparkFun-LED:LED_3MM
- D4: value (none) -> red; device SparkFun-LED:LED_5MM -> SparkFun-LED:LED_3MM
- moved LED_HEAT_CONN 34.1 mm to (43.2, 55.6), turned to 90 degrees
- moved R8 32.4 mm to (14.0, 33.0)
- moved D1 28.4 mm to (3.81, 38.1), turned to 270 degrees
- moved R9 21.0 mm to (39.4, 45.7), turned to 270 degrees
- moved LCD_CONN 19.4 mm to (43.2, 38.1)
- moved R10 12.6 mm to (39.4, 58.4), turned to 90 degrees
- moved R2 11.5 mm to (26.7, 41.9)
- moved R1 11.5 mm to (26.7, 47.0)
- moved TEMP_SENSOR_CONN 9.44 mm to (43.2, 62.5)
- moved PWR_CONN 6.73 mm to (11.4, 65.8)
- moved R5 6.48 mm to (26.7, 57.1)
- moved U$1 6.48 mm to (16.5, 33.0)
- moved R7 6.35 mm to (38.1, 27.9), turned to 180 degrees
- moved LED_COOL_CONN 5.95 mm to (43.2, 47.8)
- moved T1 5.68 mm to (24.1, 26.7)
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Connections:
- removed net BTN_DOWN: U$1.18
- removed net BTN_UP: U$1.19
- net BTN_SET: no longer U$1.20
Routing:
- net +5V: track 0.00 -> 148.8 mm
- net N$9: track 0.00 -> 92.3 mm
- net N$6: track 0.00 -> 79.2 mm
- net N$8: track 0.00 -> 64.6 mm
- net +3V3: track 0.00 -> 59.2 mm
- net N$4: track 0.00 -> 56.6 mm
- net RLY_HEAT: track 48.1 -> 93.6 mm
- net N$13: track 0.00 -> 33.3 mm
- net TEMP_DATA: track 0.00 -> 33.2 mm
- net SCL: track 0.00 -> 18.0 mm
- net BTN_COOL: track 0.00 -> 16.4 mm
- net BTN_HEAT: track 0.00 -> 16.0 mm
- net HEAT_CTRL: track 0.00 -> 15.8 mm
- net BTN_SET: track 0.00 -> 15.5 mm
- net SDA: track 0.00 -> 13.7 mm
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Other:
- board size 60.6 x 80 mm -> 55.5 x 73.7 mm
- board text added: "+"
- board text added: "+3.3v"
- board text added: "+5v"
- board text added: "-"
- board text added: "1N4148"
- board text added: "2N3904"
- board text added: "Buttons"
- board text added: "COM"
- board text added: "Cool"
- board text added: "Cool LED"
- board text added: "Data"
- board text added: "Dwn"
- board text added: "Fermentation Controller"
- board text added: "GND"
- board text added: "Heat"
- board text added: "Heat LED"
- board text added: "LCD"
- board text added: "Power"
- board text added: "Rev. 1"
- board text added: "SCL"
- board text added: "SDA"
- board text added: "Set"
- board text added: "Temp Probe"
- board text added: "Up"

Commit message: Fixed incorrect wiring for the temp probe
Parts:
- turned R3 to 0 degrees
Connections:
- removed net N$1: R3.1, U$1.15
- net +5V: now also R3.1
- net TEMP_DATA: now also U$1.15
Routing:
- net +5V: track 148.8 -> 164.6 mm
- net N$1: track 10.8 -> 0.00 mm
- net TEMP_DATA: track 33.2 -> 42.6 mm
Other:
- board text added: "Rev. 1.1"
- board text removed: "Rev. 1"
Changed lines of the file:
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@@
 <text x="4.318" y="52.578" size="0.8128" layer="21" rot="R90">Buttons</text>
 <text x="54.102" y="21.59" size="1.778" layer="21" rot="R90">Fermentation Controller</text>
-<text x="54.102" y="49.53" size="0.8128" layer="21" rot="R90">Rev. 1</text>
+<text x="54.102" y="49.276" size="0.8128" layer="21" rot="R90">Rev. 1.1</text>
 <hole x="2.286" y="71.374" drill="3.048"/>
 <hole x="53.086" y="71.374" drill="3.048"/>
@@
 <attribute name="VALUE" x="28.9306" y="42.545" size="1.27" layer="27" ratio="10" rot="R180"/>
 </element>
-<element name="R3" library="rcl" library_urn="urn:adsk.eagle:library:334" package="0207/10" package3d_urn="urn:adsk.eagle:package:23491/2" value="4.7K" x="26.67" y="52.07" smashed="yes" rot="R180">
-<attribute name="MF" value="" x="26.67" y="52.07" size="1.778" layer="27" rot="R180" display="off"/>
-<attribute name="MPN" value="" x="26.67" y="52.07" size="1.778" layer="27" rot="R180" display="off"/>
-<attribute name="OC_NEWARK" value="unknown" x="26.67" y="52.07" size="1.778" layer="27" rot="R180" display="off"/>
-<attribute name="POPULARITY" value="36" x="-5.08" y="137.16" size="1.778" layer="27" rot="R180" display="off"/>
-<attribute name="SPICEPREFIX" value="R" x="-5.08" y="137.16" size="1.778" layer="27" rot="R180" display="off"/>
-<attribute name="VALUE" x="28.9306" y="52.705" size="1.27" layer="27" ratio="10" rot="R180"/>
+<element name="R3" library="rcl" library_urn="urn:adsk.eagle:library:334" package="0207/10" package3d_urn="urn:adsk.eagle:package:23491/2" value="4.7K" x="26.67" y="52.07" smashed="yes">
+<attribute name="MF" value="" x="26.67" y="52.07" size="1.778" layer="27" display="off"/>
+<attribute name="MPN" value="" x="26.67" y="52.07" size="1.778" layer="27" display="off"/>
+<attribute name="OC_NEWARK" value="unknown" x="26.67" y="52.07" size="1.778" layer="27" display="off"/>
+<attribute name="POPULARITY" value="36" x="58.42" y="-33.02" size="1.778" layer="27" display="off"/>
+<attribute name="SPICEPREFIX" value="R" x="58.42" y="-33.02" size="1.778" layer="27" display="off"/>
+<attribute name="VALUE" x="24.4094" y="51.435" size="1.27" layer="27" ratio="10"/>
 </element>
 <element name="R5" library="rcl" library_urn="urn:adsk.eagle:library:334" package="0207/10" package3d_urn="urn:adsk.eagle:package:23491/2" value="1K" x="26.67" y="57.15" smashed="yes" rot="R180">
@@
 <wire x1="45.466" y1="51.038" x2="43.18" y2="48.752" width="0.3048" layer="1"/>
 <wire x1="43.18" y1="56.626" x2="43.18" y2="62.484" width="0.3048" layer="1"/>
+<contactref element="R3" pad="1"/>
+<wire x1="21.59" y1="52.07" x2="20.066" y2="53.594" width="0.3048" layer="16"/>
+<wire x1="20.066" y1="53.594" x2="20.066" y2="64.262" width="0.3048" layer="16"/>
+<wire x1="20.066" y1="64.262" x2="18.288" y2="66.04" width="0.3048" layer="16"/>
+<wire x1="18.288" y1="66.04" x2="17.78" y2="66.04" width="0.3048" layer="16"/>
 </signal>
 <signal name="SCL">
@@
 <contactref element="R6" pad="1"/>
 <wire x1="31.8389" y1="61.9633" x2="31.8389" y2="62.103" width="0.3048" layer="1"/>
-<wire x1="33.655" y1="60.1472" x2="31.8389" y2="61.9633" width="0.3048" layer="1"/>
-<wire x1="33.655" y1="50.7873" x2="33.655" y2="60.1472" width="0.3048" layer="1"/>
-<wire x1="34.2138" y1="50.2285" x2="33.655" y2="50.7873" width="0.3048" layer="1"/>
-<wire x1="34.2138" y1="49.3903" x2="34.2138" y2="50.2285" width="0.3048" layer="1"/>
-<wire x1="35.4711" y1="48.133" x2="34.2138" y2="49.3903" width="0.3048" layer="1"/>
+<wire x1="31.8389" y1="61.9633" x2="33.655" y2="60.1472" width="0.3048" layer="1"/>
 <wire x1="31.8389" y1="62.103" x2="31.75" y2="62.23" width="0.3048" layer="1"/>
-<wire x1="35.4711" y1="48.133" x2="35.56" y2="48.26" width="0.3048" layer="1"/>
+<wire x1="33.655" y1="50.165" x2="35.56" y2="48.26" width="0.3048" layer="1"/>
+<wire x1="33.655" y1="60.1472" x2="33.655" y2="50.165" width="0.3048" layer="1"/>
 </signal>
 <signal name="BTN_SET">
@@
 <wire x1="17.7292" y1="43.2435" x2="17.78" y2="43.18" width="0.3048" layer="16"/>
 </signal>
-<signal name="N$1">
+<signal name="TEMP_DATA">
+<contactref element="TEMP_SENSOR_CONN" pad="3"/>
 <contactref element="U$1" pad="15"/>
-<contactref element="R3" pad="1"/>
-<wire x1="31.8389" y1="51.7652" x2="31.8389" y2="52.0446" width="0.3048" layer="1"/>
-<wire x1="33.655" y1="49.9491" x2="31.8389" y2="51.7652" width="0.3048" layer="1"/>
-<wire x1="33.655" y1="44.6405" x2="33.655" y2="49.9491" width="0.3048" layer="1"/>
-<wire x1="34.4932" y1="43.8023" x2="33.655" y2="44.6405" width="0.3048" layer="1"/>
-<wire x1="34.6329" y1="43.8023" x2="34.4932" y2="43.8023" width="0.3048" layer="1"/>
-<wire x1="35.1917" y1="43.2435" x2="34.6329" y2="43.8023" width="0.3048" layer="1"/>
-<wire x1="35.4711" y1="43.2435" x2="35.1917" y2="43.2435" width="0.3048" layer="1"/>
-<wire x1="31.8389" y1="52.0446" x2="31.75" y2="52.07" width="0.3048" layer="1"/>
-<wire x1="35.4711" y1="43.2435" x2="35.56" y2="43.18" width="0.3048" layer="1"/>
-</signal>
-<signal name="TEMP_DATA">
 <contactref element="R3" pad="2"/>
-<contactref element="TEMP_SENSOR_CONN" pad="3"/>
-<wire x1="25.1333" y1="60.9854" x2="33.5026" y2="69.3547" width="0.3048" layer="1"/>
-<wire x1="25.1333" y1="56.7436" x2="25.1333" y2="60.9854" width="0.3048" layer="1"/>
-<wire x1="21.5011" y1="53.1114" x2="25.1333" y2="56.7436" width="0.3048" layer="1"/>
-<wire x1="21.5011" y1="52.1843" x2="21.5011" y2="53.1114" width="0.3048" layer="1"/>
-<wire x1="21.5011" y1="52.1843" x2="21.59" y2="52.07" width="0.3048" layer="1"/>
-<wire x1="40.3093" y1="69.3547" x2="43.18" y2="66.484" width="0.3048" layer="1"/>
-<wire x1="33.5026" y1="69.3547" x2="40.3093" y2="69.3547" width="0.3048" layer="1"/>
+<wire x1="31.75" y1="52.07" x2="31.75" y2="49.276" width="0.3048" layer="1"/>
+<wire x1="31.75" y1="49.276" x2="33.528" y2="47.498" width="0.3048" layer="1"/>
+<wire x1="33.528" y1="47.498" x2="33.528" y2="44.958" width="0.3048" layer="1"/>
+<wire x1="33.528" y1="44.958" x2="35.306" y2="43.18" width="0.3048" layer="1"/>
+<wire x1="35.306" y1="43.18" x2="35.56" y2="43.18" width="0.3048" layer="1"/>
+<wire x1="31.75" y1="52.07" x2="28.956" y2="54.864" width="0.3048" layer="1"/>
+<wire x1="28.956" y1="54.864" x2="28.956" y2="66.548" width="0.3048" layer="1"/>
+<wire x1="28.956" y1="66.548" x2="31.496" y2="69.088" width="0.3048" layer="1"/>
+<wire x1="40.576" y1="69.088" x2="43.18" y2="66.484" width="0.3048" layer="1"/>
+<wire x1="31.496" y1="69.088" x2="40.576" y2="69.088" width="0.3048" layer="1"/>
 </signal>
 <signal name="N$13">
