File: drawings/eagle/module.sch (EAGLE design)
At the start: 25 parts, among them T1 2N3904, T2 2N3904

Commit message: Finished rev1 of the circuit board and moved to a drawings directory
Parts:
- BUTTON_CONN, LCD_CONN: MF (none) -> JST (JAPAN SOLDERLESS TERMINALS); MPN (none) -> S4B-PH-K-S (LF)(SN); OC_NEWARK (none) -> 38K8074
- D1, D2: MF (none) -> MULTICOMP PRO; MPN (none) -> 1N4148 (DO-35); OC_NEWARK (none) -> 05AC0533
- D3: value (none) -> blue; device SparkFun-LED:LED5MM -> SparkFun-LED:LED3MM; MF (none) -> VISHAY; MPN (none) -> TLHB4400; OC_NEWARK (none) -> 09X0596
- D4: value (none) -> red; device SparkFun-LED:LED5MM -> SparkFun-LED:LED3MM; MF (none) -> VCC (VISUAL COMMUNICATIONS COMPANY); MPN (none) -> 4300F1LC; OC_NEWARK (none) -> 05C1482
- LED_COOL_CONN, LED_HEAT_CONN, PWR_CONN: MF (none) -> JST (JAPAN SOLDERLESS TERMINALS); MPN (none) -> S2B-PH-K-S (LF)(SN); OC_NEWARK (none) -> 38K8066
- R1, R10, R2, R3, R5, R6, R7, R8, R9, R_COOL, R_HEAT, SWITCHED_PWR_BLOCK: OC_NEWARK (none) -> unknown
- T1, T2: MF (none) -> ONSEMI; MPN (none) -> 2N3904TF; OC_NEWARK (none) -> 05R0381
- TEMP_SENSOR_CONN: MF (none) -> JST (JAPAN SOLDERLESS TERMINALS); MPN (none) -> S3B-PH-K-S (LF)(SN); OC_NEWARK (none) -> 38K8070
- U$1: MF (none) -> PARTICLE; MPN (none) -> PHOTONH; OC_NEWARK (none) -> 60AC3758
Connections:
- removed net BTN_DOWN: U$1.D5
- removed net BTN_UP: U$1.D6
- net BTN_SET: no longer U$1.D7
Other:
- moved on the sheet: D3

Commit message: Fixed incorrect wiring for the temp probe
Connections:
- removed net N$1: R3.1, U$1.D2
- net +5V: now also R3.1
- net TEMP_DATA: now also U$1.D2
Other:
- moved on the sheet: R3
Changed lines of the file:
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@@
 <attribute name="OC_NEWARK" value="05C1482"/>
 </part>
+<part name="P+11" library="supply1" library_urn="urn:adsk.eagle:library:371" deviceset="+5V" device=""/>
 </parts>
 <sheets>
@@
 <attribute name="MPN" x="106.68" y="88.9" size="1.778" layer="96" display="off"/>
 </instance>
-<instance part="R3" gate="G$1" x="104.14" y="99.06" smashed="yes">
-<attribute name="NAME" x="100.33" y="100.5586" size="1.778" layer="95"/>
-<attribute name="VALUE" x="100.33" y="95.758" size="1.778" layer="96"/>
-<attribute name="OC_NEWARK" x="104.14" y="99.06" size="1.778" layer="96" display="off"/>
-<attribute name="MF" x="104.14" y="99.06" size="1.778" layer="96" display="off"/>
-<attribute name="MPN" x="104.14" y="99.06" size="1.778" layer="96" display="off"/>
+<instance part="R3" gate="G$1" x="152.4" y="99.06" smashed="yes" rot="R90">
+<attribute name="NAME" x="150.9014" y="95.25" size="1.778" layer="95" rot="R90"/>
+<attribute name="VALUE" x="155.702" y="95.25" size="1.778" layer="96" rot="R90"/>
+<attribute name="OC_NEWARK" x="152.4" y="99.06" size="1.778" layer="96" rot="R90" display="off"/>
+<attribute name="MF" x="152.4" y="99.06" size="1.778" layer="96" rot="R90" display="off"/>
+<attribute name="MPN" x="152.4" y="99.06" size="1.778" layer="96" rot="R90" display="off"/>
 </instance>
 <instance part="GND1" gate="1" x="53.34" y="139.7" smashed="yes" rot="R270">
@@
 <attribute name="VALUE" x="149.86" y="116.84" size="1.778" layer="96" rot="R90"/>
 </instance>
-<instance part="GND6" gate="1" x="149.86" y="111.76" smashed="yes" rot="R270">
-<attribute name="VALUE" x="147.32" y="114.3" size="1.778" layer="96" rot="R270"/>
+<instance part="GND6" gate="1" x="144.78" y="111.76" smashed="yes" rot="R270">
+<attribute name="VALUE" x="142.24" y="114.3" size="1.778" layer="96" rot="R270"/>
 </instance>
 <instance part="R_COOL" gate="G$1" x="48.26" y="60.96" smashed="yes">
@@
 <attribute name="MF" x="137.16" y="66.04" size="1.778" layer="96" display="off"/>
 <attribute name="MPN" x="137.16" y="66.04" size="1.778" layer="96" display="off"/>
+</instance>
+<instance part="P+11" gate="1" x="152.4" y="88.9" smashed="yes" rot="R180">
+<attribute name="VALUE" x="154.94" y="93.98" size="1.778" layer="96" rot="R270"/>
 </instance>
 </instances>
@@
 <segment>
 <pinref part="TEMP_SENSOR_CONN" gate="G$1" pin="2"/>
-<wire x1="154.94" y1="111.76" x2="152.4" y2="111.76" width="0.1524" layer="91"/>
+<wire x1="154.94" y1="111.76" x2="147.32" y2="111.76" width="0.1524" layer="91"/>
 <pinref part="GND6" gate="1" pin="GND"/>
 </segment>
@@
 <wire x1="17.78" y1="139.7" x2="20.32" y2="139.7" width="0.1524" layer="91"/>
 <wire x1="20.32" y1="139.7" x2="20.32" y2="137.16" width="0.1524" layer="91"/>
+</segment>
+<segment>
+<pinref part="R3" gate="G$1" pin="1"/>
+<wire x1="152.4" y1="93.98" x2="152.4" y2="91.44" width="0.1524" layer="91"/>
+<pinref part="P+11" gate="1" pin="+5V"/>
 </segment>
 </net>
@@
 </segment>
 </net>
-<net name="N$1" class="0">
+<net name="TEMP_DATA" class="0">
+<segment>
+<pinref part="TEMP_SENSOR_CONN" gate="G$1" pin="3"/>
+<label x="147.32" y="109.22" size="1.778" layer="95" rot="R270" xref="yes"/>
+<wire x1="154.94" y1="109.22" x2="152.4" y2="109.22" width="0.1524" layer="91"/>
+<junction x="152.4" y="109.22"/>
+<wire x1="152.4" y1="109.22" x2="147.32" y2="109.22" width="0.1524" layer="91"/>
+<pinref part="R3" gate="G$1" pin="2"/>
+<wire x1="152.4" y1="104.14" x2="152.4" y2="109.22" width="0.1524" layer="91"/>
+</segment>
 <segment>
 <pinref part="U$1" gate="G$1" pin="D2"/>
-<pinref part="R3" gate="G$1" pin="1"/>
-<wire x1="99.06" y1="99.06" x2="96.52" y2="99.06" width="0.1524" layer="91"/>
-</segment>
-</net>
-<net name="TEMP_DATA" class="0">
-<segment>
-<pinref part="R3" gate="G$1" pin="2"/>
-<wire x1="109.22" y1="99.06" x2="111.76" y2="99.06" width="0.1524" layer="91"/>
-<label x="111.76" y="99.06" size="1.778" layer="95" xref="yes"/>
-</segment>
-<segment>
-<pinref part="TEMP_SENSOR_CONN" gate="G$1" pin="3"/>
-<wire x1="154.94" y1="109.22" x2="152.4" y2="109.22" width="0.1524" layer="91"/>
-<label x="152.4" y="109.22" size="1.778" layer="95" rot="R270" xref="yes"/>
-</segment>
-</net>
+<wire x1="96.52" y1="99.06" x2="99.06" y2="99.06" width="0.1524" layer="91"/>
+<label x="99.06" y="99.06" size="1.778" layer="95" xref="yes"/>
+</segment>
+</net>
